File: implementation/USB_UART.kicad_sch (KiCad schematic)
At the start: 16 parts, among them J7 USB_B_Micro, U2 CP2102N-Axx-xQFN28

Commit message: add Pin Socket for CamDroid (J8); rerouted, gerber created
Parts:
- Q5, Q6: renamed from Q?; footprint Package_TO_SOT_SMD:SOT-23_Handsoldering -> Package_TO_SOT_SMD:SOT-23; symbol Device:Q_NPN_BEC -> Transistor_BJT:SS8050
- TP7: renamed from TP?; now left out of the parts list
- gave numbers to parts that had none: 8
